File: Totebox Alert V3/Totebox Alert.kicad_pcb (KiCad board)
At the start: 2 copper layers, 175 x 95 mm, 49 parts, among them J1 Optocoupler In, J12 Boost Conv. Out, J2 Buzzer, J3 Optocoupler Out, J4 SMPS IN, J5 AC, J8 SMPS OUT, J9 Boost Conv. In, SW1 SW_SPST, U3 ESP32-DEVKITC-32UE

Commit message: add esp32 auto reset capabilities on both ground and floor units
Parts:
- 220 VAC: renamed from J5
- BC IN: renamed from J9
- BC OUT: renamed from J12
- Push Button: renamed from SW1
- SMPS IN: renamed from J4
- SMPS OUT: renamed from J8
- renumbered J2 to Buzzer, F1 to FUSE, D1 to LED
Changed lines of the file:
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@@
 		(descr "Terminal Block Phoenix MKDS-1,5-3-5.08, 3 pins, pitch 5.08mm, size 15.2x9.8mm^2, drill diamater 1.3mm, pad diameter 2.6mm, see http://www.farnell.com/datasheets/100425.pdf, script-generated using https://github.com/pointhi/kicad-footprint-generator/scripts/TerminalBlock_Phoenix")
 		(tags "THT Terminal Block Phoenix MKDS-1,5-3-5.08 pitch 5.08mm size 15.2x9.8mm^2 drill 1.3mm pad 2.6mm")
-		(property "Reference" "J5"
-			(at 5.08 -6.26 0)
+		(property "Reference" "220 VAC"
+			(at 5 -3.72 0)
 			(layer "F.SilkS")
 			(effects
@@
 		(descr "Terminal Block Phoenix MKDS-1,5-3-5.08, 3 pins, pitch 5.08mm, size 15.2x9.8mm^2, drill diamater 1.3mm, pad diameter 2.6mm, see http://www.farnell.com/datasheets/100425.pdf, script-generated using https://github.com/pointhi/kicad-footprint-generator/scripts/TerminalBlock_Phoenix")
 		(tags "THT Terminal Block Phoenix MKDS-1,5-3-5.08 pitch 5.08mm size 15.2x9.8mm^2 drill 1.3mm pad 2.6mm")
-		(property "Reference" "J4"
-			(at 5.08 -6.26 0)
+		(property "Reference" "SMPS IN"
+			(at 5.06 -3.57 0)
 			(layer "F.SilkS")
 			(effects
@@
 		(descr "JST XH series connector, B3B-XH-A (http://www.jst-mfg.com/product/pdf/eng/eXH.pdf), generated with kicad-footprint-generator")
 		(tags "connector JST XH vertical")
-		(property "Reference" "J2"
+		(property "Reference" "Buzzer"
 			(at 2.5 -3.55 0)
 			(layer "F.SilkS")
@@
 		(descr "Terminal Block Phoenix MKDS-1,5-2-5.08, 2 pins, pitch 5.08mm, size 10.2x9.8mm^2, drill diamater 1.3mm, pad diameter 2.6mm, see http://www.farnell.com/datasheets/100425.pdf, script-generated using https://github.com/pointhi/kicad-footprint-generator/scripts/TerminalBlock_Phoenix")
 		(tags "THT Terminal Block Phoenix MKDS-1,5-2-5.08 pitch 5.08mm size 10.2x9.8mm^2 drill 1.3mm pad 2.6mm")
-		(property "Reference" "J12"
+		(property "Reference" "BC OUT"
 			(at 2.54 -6.26 90)
 			(layer "F.SilkS")
@@
 		(descr "Terminal Block Phoenix MKDS-1,5-2-5.08, 2 pins, pitch 5.08mm, size 10.2x9.8mm^2, drill diamater 1.3mm, pad diameter 2.6mm, see http://www.farnell.com/datasheets/100425.pdf, script-generated using https://github.com/pointhi/kicad-footprint-generator/scripts/TerminalBlock_Phoenix")
 		(tags "THT Terminal Block Phoenix MKDS-1,5-2-5.08 pitch 5.08mm size 10.2x9.8mm^2 drill 1.3mm pad 2.6mm")
-		(property "Reference" "D1"
+		(property "Reference" "LED"
 			(at 2.54 -6.26 0)
 			(layer "F.SilkS")
@@
 		(descr "Terminal Block Phoenix MKDS-1,5-2-5.08, 2 pins, pitch 5.08mm, size 10.2x9.8mm^2, drill diamater 1.3mm, pad diameter 2.6mm, see http://www.farnell.com/datasheets/100425.pdf, script-generated using https://github.com/pointhi/kicad-footprint-generator/scripts/TerminalBlock_Phoenix")
 		(tags "THT Terminal Block Phoenix MKDS-1,5-2-5.08 pitch 5.08mm size 10.2x9.8mm^2 drill 1.3mm pad 2.6mm")
-		(property "Reference" "J8"
-			(at 2.54 -6.26 180)
+		(property "Reference" "SMPS OUT"
+			(at 2.59 -4.05 180)
 			(layer "F.SilkS")
 			(effects
@@
 		(descr "Terminal Block Phoenix MKDS-1,5-2-5.08, 2 pins, pitch 5.08mm, size 10.2x9.8mm^2, drill diamater 1.3mm, pad diameter 2.6mm, see http://www.farnell.com/datasheets/100425.pdf, script-generated using https://github.com/pointhi/kicad-footprint-generator/scripts/TerminalBlock_Phoenix")
 		(tags "THT Terminal Block Phoenix MKDS-1,5-2-5.08 pitch 5.08mm size 10.2x9.8mm^2 drill 1.3mm pad 2.6mm")
-		(property "Reference" "J9"
-			(at 2.54 -6.26 90)
+		(property "Reference" "BC IN"
+			(at 2.6 -3.97 90)
 			(layer "F.SilkS")
 			(effects
@@
 		(descr "Terminal Block Phoenix MKDS-1,5-2-5.08, 2 pins, pitch 5.08mm, size 10.2x9.8mm^2, drill diamater 1.3mm, pad diameter 2.6mm, see http://www.farnell.com/datasheets/100425.pdf, script-generated using https://github.com/pointhi/kicad-footprint-generator/scripts/TerminalBlock_Phoenix")
 		(tags "THT Terminal Block Phoenix MKDS-1,5-2-5.08 pitch 5.08mm size 10.2x9.8mm^2 drill 1.3mm pad 2.6mm")
-		(property "Reference" "SW1"
+		(property "Reference" "Push Button"
 			(at 2.54 -6.26 0)
 			(layer "F.SilkS")
@@
 		(descr "Fuseholder horizontal open, 5x20mm, 500V, 16A, Schurter 0031.8201, https://us.schurter.com/bundles/snceschurter/epim/_ProdPool_/newDS/en/typ_OGN.pdf")
 		(tags "Fuseholder horizontal open 5x20 Schurter 0031.8201")
-		(property "Reference" "F1"
+		(property "Reference" "FUSE"
 			(at 10.8 -0.2 90)
 			(layer "F.SilkS")
